Commit message: First iteration of HWIs: DC, CCD, Diode, Fixing Laser, CCD Custom Controller, Laser & Diode GPIO Controllers

File: src/description/ros2_control/science/science.sensor_diode.ros2_control.xacro (robot description, xacro)
@@ -1,16 +1,16 @@
 <?xml version="1.0"?>
 <robot xmlns:xacro="http://www.ros.org/wiki/xacro">
-    <xacro:macro name="laser_ros2_control" params="name can_interface:=can0 port_id:=0">
+    <xacro:macro name="sensor_diode_ros2_control" params="name can_interface:=can0">
         <ros2_control name="${name}" type="system">
             <hardware>
-                <plugin>laser_ros2_control/LaserHardwareInterface</plugin>
+                <plugin>sensor_diode_ros2_control/SensorDiodeHardwareInterface</plugin>
                 <param name="can_interface">${can_interface}</param>
-                <param name="can_id">0x130</param>
-                <param name="port_id">${port_id}</param>
+                <param name="can_id">0x110</param>
             </hardware>
             <gpio name="${name}">
-                <state_interface name="laser_state"/>
+                <state_interface name="wavelength_intensity"/>
+                <state_interface name="command_success"/>
                 <state_interface name="is_connected"/>
-                <command_interface name="laser_command"/>
+                <command_interface name="request_measurement"/>
             </gpio>
         </ros2_control>

File: src/description/urdf/athena_science.urdf.xacro (robot description, xacro)
@@ -9,4 +9,6 @@
   <xacro:include filename="$(find description)/ros2_control/science/science.talon.ros2_control.xacro"/>
   <xacro:include filename="$(find description)/ros2_control/science/science.laser.ros2_control.xacro"/>
+  <xacro:include filename="$(find description)/ros2_control/science/science.ccd.ros2_control.xacro"/>
+  <xacro:include filename="$(find description)/ros2_control/science/science.sensor_diode.ros2_control.xacro"/>
   <!-- create link fixed to the "world" -->
   <link name="world"/>
@@ -25,7 +27,11 @@
     <xacro:dc_ros2_control name="dc"/>
     <!-- Import talon ros2_control description -->
-    <xacro:talon_ros2_control name="talon"/>
+    <!-- <xacro:talon_ros2_control name="talon"/> -->
     <!-- Import laser ros2_control description (CAN-based) -->
     <xacro:laser_ros2_control name="spectrometry_laser"/>
+    <!-- Import CCD ros2_control description (CAN-based) -->
+    <xacro:ccd_ros2_control name="spectrometry_ccd"/>
+    <!-- Import sensor diode ros2_control description (CAN-based) -->
+    <xacro:sensor_diode_ros2_control name="sensor_diode"/>
   </xacro:unless>
 </robot>
