Commit message: HWI Upgrades (#110)
* changed broadcaster to controller and included other telemetry information

* odrive upgrades

* added request services

* included status decoding in RMDs

* decode error value and warn/error out depending on response

* reformatted rmd HWI

* saving some one shot progress

* encoding and decoding across command interfaces seems to be working

* holy fucking shit it works. Need to implement Torque control and then start doing doing this implementation on the rest of the HWIs

* updated smc hwi, issue with servo hwi

* fixed state issue, accepts all state interfaces and filters accordingly

* saving progress, killswitch seems to not be sending can messages for some reason

* saving changes, for some reason I cant see power module can commands being sent

* Power module and SMCs seem to be working, initial implementation of LED HWI created

* led hwi looks like its working

* added limit switch and rotary encoder HWI, included all necessary HWIs, needs fixing

* fixed motor status controller, manually choose command and state interfaces if default don't apply

* 3dof specific fixes

* motor status controller includes gpios, removing unnecessary gpio controllers

* Added DC Motor HWI

* Small changes to DC Motor HWI

* Fixing HWI issue

* Small Fix

* First test for steppers

* Moved revised athena_science code to monorepo

* Fixing Science Controller + HWI Templates for Steppers & Servos

* Restore accidentally deleted science.mock.ros2_control.xacro

* stepper stuff like kinda works??

* implemented and tested in virtual can servo, stepper, and dc HWIs

* working arm and steppers/DC motors

* WORKING DRIVE AND ARM

* quick fixes (joystick_index not set and removing /vscode and .codex

---------

Co-authored-by: duttaishan01 <duttaishan01@FIGARO.myguest.virtualbox.org>
Co-authored-by: HGardiner1 <henrygdnr@gmail.com>
Co-authored-by: UMDLoop Jetson Orin NX <umdloop@gmail.com>

File: src/description/ros2_control/arm/arm.rmd.ros2_control.xacro (robot description, xacro)
@@ -8,5 +8,5 @@
         <param name="logger_rate">5</param> <!-- Hz -->
         <param name="logger_state">0</param> <!-- 0 for off, 1 for on -->
-        <param name="can_interface">can0</param>
+        <param name="can_interface">can1</param>
       </hardware>
       <joint name="shoulder_pitch">
@@ -15,8 +15,16 @@
         <param name="joint_orientation">1.0</param>
         <param name="operating_velocity">150</param> <!-- motor dps -->
+        <command_interface name="position" />
+        <command_interface name="velocity"/>
+        <command_interface name="status_request"/>
+        <command_interface name="maintenance_request"/>
+        <command_interface name="maintenance_frame_high"/>
+        <command_interface name="maintenance_frame_low"/>
+        <command_interface name="maintenance_data_count"/>
         <state_interface name="position"/>
         <state_interface name="velocity"/>
         <state_interface name="motor_temperature"/>
         <state_interface name="torque_current"/>
+        <state_interface name="status"/>
       </joint>
       <joint name="elbow_pitch">
@@ -25,8 +33,16 @@
         <param name="joint_orientation">-1.0</param>
         <param name="operating_velocity">150</param> <!-- motor dps -->
+        <command_interface name="position" />
+        <command_interface name="velocity"/>
+        <command_interface name="status_request"/>
+        <command_interface name="maintenance_request"/>
+        <command_interface name="maintenance_frame_high"/>
+        <command_interface name="maintenance_frame_low"/>
+        <command_interface name="maintenance_data_count"/>
         <state_interface name="position"/>
         <state_interface name="velocity"/>
         <state_interface name="motor_temperature"/>
         <state_interface name="torque_current"/>
+        <state_interface name="status"/>
       </joint>
     </ros2_control>

File: src/description/ros2_control/arm/arm.servo.ros2_control.xacro (robot description, xacro)
@@ -8,5 +8,5 @@
                 <param name="logger_rate">5</param> <!-- Hz -->
                 <param name="logger_state">0</param> <!-- 0 for off, 1 for on -->
-                <param name="can_interface">can0</param>
+                <param name="can_interface">can1</param>
                 <param name="can_id">0x80</param>
             </hardware>
@@ -20,5 +20,46 @@
                 <command_interface name="position" />
                 <command_interface name="velocity"/>
-                <state_interface name="position" />
+                <command_interface name="status_request"/>
+                <command_interface name="maintenance_request"/>
+                <command_interface name="maintenance_frame_high"/>
+                <command_interface name="maintenance_frame_low"/>
+                <command_interface name="maintenance_data_count"/>
+                <state_interface name="position"/>
+                <state_interface name="velocity"/>
+                <state_interface name="status"/>
+            </joint>
+            <joint name="cam_0">
+                <param name="node_id">0x2</param>
+                <param name="gear_ratio">1</param>
+                <param name="max_pos">180</param> <!-- degrees -->
+                <param name="servo_type">standard</param> <!-- standard or continuous -->
+                <param name="joint_type">revolute</param> <!-- revolute or prismatic -->
+                <command_interface name="position" />
+                <command_interface name="velocity"/>
+                <command_interface name="status_request"/>
+                <command_interface name="maintenance_request"/>
+                <command_interface name="maintenance_frame_high"/>
+                <command_interface name="maintenance_frame_low"/>
+                <command_interface name="maintenance_data_count"/>
+                <state_interface name="position"/>
+                <state_interface name="velocity"/>
+                <state_interface name="status"/>
+            </joint>
+            <joint name="cam_1">
+                <param name="node_id">0x3</param>
+                <param name="gear_ratio">1</param>
+                <param name="max_pos">180</param> <!-- degrees -->
+                <param name="servo_type">standard</param> <!-- standard or continuous -->
+                <param name="joint_type">revolute</param> <!-- revolute or prismatic -->
+                <command_interface name="position" />
+                <command_interface name="velocity"/>
+                <command_interface name="status_request"/>
+                <command_interface name="maintenance_request"/>
+                <command_interface name="maintenance_frame_high"/>
+                <command_interface name="maintenance_frame_low"/>
+                <command_interface name="maintenance_data_count"/>
+                <state_interface name="position"/>
+                <state_interface name="velocity"/>
+                <state_interface name="status"/>
             </joint>
         </ros2_control>

File: src/description/ros2_control/arm/arm.smc_2dof.ros2_control.xacro (robot description, xacro)
@@ -8,5 +8,5 @@
         <param name="logger_rate">5</param> <!-- Hz -->
         <param name="logger_state">0</param> <!-- 0 for off, 1 for on -->
-        <param name="can_interface">can0</param>
+        <param name="can_interface">can1</param>
       </hardware>
       <joint name="base_yaw">
@@ -17,10 +17,34 @@
         <command_interface name="position"/>
         <command_interface name="velocity"/>
+        <command_interface name="status_request"/>
+        <command_interface name="maintenance_request"/>
+        <command_interface name="maintenance_frame_high"/>
+        <command_interface name="maintenance_frame_low"/>
+        <command_interface name="maintenance_data_count"/>
         <state_interface name="position"/>
         <state_interface name="velocity"/>
         <state_interface name="motor_temperature"/>
         <state_interface name="torque_current"/>
+        <state_interface name="status"/>
       </joint>
       <joint name="wrist_pitch">
+        <param name="node_id">0x147</param>
+        <param name="gear_ratio">40</param>
+        <param name="joint_orientation">1.0</param>
+        <param name="operating_velocity">1000</param> <!-- motor dps -->
+        <command_interface name="position"/>
+        <command_interface name="velocity"/>
+        <command_interface name="status_request"/>
+        <command_interface name="maintenance_request"/>
+        <command_interface name="maintenance_frame_high"/>
+        <command_interface name="maintenance_frame_low"/>
+        <command_interface name="maintenance_data_count"/>
+        <state_interface name="position"/>
+        <state_interface name="velocity"/>
+        <state_interface name="motor_temperature"/>
+        <state_interface name="torque_current"/>
+        <state_interface name="status"/>
+      </joint>
+      <joint name="wrist_roll">
         <param name="node_id">0x145</param>
         <param name="gear_ratio">40</param>
@@ -29,20 +53,14 @@
         <command_interface name="position"/>
         <command_interface name="velocity"/>
+        <command_interface name="status_request"/>
+        <command_interface name="maintenance_request"/>
+        <command_interface name="maintenance_frame_high"/>
+        <command_interface name="maintenance_frame_low"/>
+        <command_interface name="maintenance_data_count"/>
         <state_interface name="position"/>
         <state_interface name="velocity"/>
         <state_interface name="motor_temperature"/>
         <state_interface name="torque_current"/>
-      </joint>
-      <joint name="wrist_roll">
-        <param name="node_id">0x147</param>
-        <param name="gear_ratio">40</param>
-        <param name="joint_orientation">1.0</param>
-        <param name="operating_velocity">1000</param> <!-- motor dps -->
-        <command_interface name="position"/>
-        <command_interface name="velocity"/>
-        <state_interface name="position"/>
-        <state_interface name="velocity"/>
-        <state_interface name="motor_temperature"/>
-        <state_interface name="torque_current"/>
+        <state_interface name="status"/>
       </joint>
     </ros2_control>

File: src/description/ros2_control/arm/arm.smc_3dof.ros2_control.xacro (robot description, xacro)
@@ -8,5 +8,5 @@
         <param name="logger_rate">5</param> <!-- Hz -->
         <param name="logger_state">0</param> <!-- 0 for off, 1 for on -->
-        <param name="can_interface">can0</param>
+        <param name="can_interface">can1</param>
       </hardware>
       <joint name="base_yaw">
@@ -17,8 +17,14 @@
         <command_interface name="position"/>
         <command_interface name="velocity"/>
+        <command_interface name="status_request"/>
+        <command_interface name="maintenance_request"/>
+        <command_interface name="maintenance_frame_high"/>
+        <command_interface name="maintenance_frame_low"/>
+        <command_interface name="maintenance_data_count"/>
         <state_interface name="position"/>
         <state_interface name="velocity"/>
         <state_interface name="motor_temperature"/>
         <state_interface name="torque_current"/>
+        <state_interface name="status"/>
       </joint>
     </ros2_control>

File: src/description/ros2_control/arm/arm.talon_2dof.ros2_control.xacro (robot description, xacro)
@@ -13,5 +13,5 @@
           <param name="logger_rate">5</param> <!-- Hz -->
           <param name="logger_state">0</param> <!-- 0 for off, 1 for on -->
-          <param name="can_interface">can0</param>
+          <param name="can_interface">can1</param>
         </xacro:unless>
       </hardware>
@@ -32,6 +32,10 @@
         <command_interface name="position"/>
         <command_interface name="velocity"/>
+        <command_interface name="status_request"/>
         <state_interface name="position"/>
         <state_interface name="velocity"/>
+        <state_interface name="motor_temperature"/>
+        <state_interface name="torque_current"/>
+        <state_interface name="status"/>
       </joint>
     </ros2_control>

File: src/description/ros2_control/arm/arm.talon_3dof.ros2_control.xacro (robot description, xacro)
@@ -12,5 +12,5 @@
           <param name="logger_rate">5</param> <!-- Hz -->
           <param name="logger_state">0</param> <!-- 0 for off, 1 for on -->
-          <param name="can_interface">can0</param>
+          <param name="can_interface">can1</param>
         </xacro:unless>
       </hardware>
@@ -30,8 +30,10 @@
         <command_interface name="position"/>
         <command_interface name="velocity"/>
+        <command_interface name="status_request"/>
         <state_interface name="position"/>
         <state_interface name="velocity"/>
         <state_interface name="motor_temperature"/>
         <state_interface name="torque_current"/>
+        <state_interface name="status"/>
       </joint>
       <joint name="wrist_motor_b">
@@ -50,8 +52,10 @@
         <command_interface name="position"/>
         <command_interface name="velocity"/>
+        <command_interface name="status_request"/>
         <state_interface name="position"/>
         <state_interface name="velocity"/>
         <state_interface name="motor_temperature"/>
         <state_interface name="torque_current"/>
+        <state_interface name="status"/>
       </joint>
       <joint name="wrist_motor_c">
@@ -70,8 +74,10 @@
         <command_interface name="position"/>
         <command_interface name="velocity"/>
+        <command_interface name="status_request"/>
         <state_interface name="position"/>
         <state_interface name="velocity"/>
         <state_interface name="motor_temperature"/>
         <state_interface name="torque_current"/>
+        <state_interface name="status"/>
       </joint>
       <joint name="gripper_claw">
@@ -91,6 +97,10 @@
         <command_interface name="position"/>
         <command_interface name="velocity"/>
+        <command_interface name="status_request"/>
         <state_interface name="position"/>
         <state_interface name="velocity"/>
+        <state_interface name="motor_temperature"/>
+        <state_interface name="torque_current"/>
+        <state_interface name="status"/>
       </joint>
     </ros2_control>

File: src/description/ros2_control/drive/drive.led.ros2_control.xacro (robot description, xacro)
@@ -1,15 +1,23 @@
 <?xml version="1.0"?>
 <robot xmlns:xacro="http://www.ros.org/wiki/xacro">
-  <xacro:macro name="led_ros2_control" params="name gpio_pin default_state:=off">
+  <xacro:macro name="led_ros2_control" params="name can_interface">
     <ros2_control name="${name}" type="system">
       <hardware>
         <plugin>led_ros2_control/LEDHardwareInterface</plugin>
-        <param name="gpio_pin">${gpio_pin}</param>
-        <param name="default_state">${default_state}</param>
+        <param name="can_interface">${can_interface}</param>
+        <param name="can_id">0x120</param>
+        <param name="update_rate">10</param> <!-- Hz -->
+        <param name="logger_rate">5</param> <!-- Hz -->
+        <param name="logger_state">0</param> <!-- 0 for off, 1 for on -->
       </hardware>
       <gpio name="${name}">
-        <state_interface name="led_state"/>
-        <state_interface name="is_connected"/>
-        <command_interface name="led_command"/>
+        <param name="is_rgb">true</param>
+        <param name="node_id">0</param>
+        <state_interface name="status"/>
+        <command_interface name="red"/>
+        <command_interface name="green"/>
+        <command_interface name="blue"/>
+        <!-- <command_interface name="intensity"/> -->
+        <command_interface name="status_request"/>
       </gpio>
     </ros2_control>

File: src/description/ros2_control/drive/drive.odrive.ros2_control.xacro (robot description, xacro)
@@ -1,9 +1,18 @@
 <?xml version="1.0"?>
 <robot xmlns:xacro="http://www.ros.org/wiki/xacro">
-  <xacro:macro name="odrive_ros2_control" params="name">
+  <xacro:macro name="odrive_ros2_control" params="name deactivate_odrive">
     <ros2_control name="${name}" type="system">
       <hardware>
-        <plugin>odrive_ros2_control_plugin/ODriveHardwareInterface</plugin>
-        <param name="can">can1</param>
+        <param name="deactivate_odrive">${deactivate_odrive}</param>
+        <xacro:if value="${deactivate_odrive}">
+          <plugin>mock_components/GenericSystem</plugin>
+        </xacro:if>
+        <xacro:unless value="${deactivate_odrive}">
+          <plugin>odrive_ros2_control_plugin/ODriveHardwareInterface</plugin>
+          <param name="update_rate">30</param> <!-- Hz -->
+          <param name="logger_rate">5</param> <!-- Hz -->
+          <param name="logger_state">0</param> <!-- 0 for off, 1 for on -->
+          <param name="can">can1</param>
+        </xacro:unless>
       </hardware>
       <joint name="steer_bl_joint">
@@ -12,8 +21,11 @@
         <command_interface name="position"/>
         <command_interface name="velocity"/>
-        <state_interface name="position">
-          <param name="initial_value">0.0</param>
-        </state_interface>
+        <!-- <command_interface name="status_request"/>
+        <command_interface name="maintenance_request"/> -->
+        <state_interface name="position"/>
         <state_interface name="velocity"/>
+        <state_interface name="motor_temperature"/>
+        <state_interface name="torque_current"/>
+        <!-- <state_interface name="status"/> -->
       </joint>
       <joint name="steer_br_joint">
@@ -22,8 +34,11 @@
         <command_interface name="position"/>
         <command_interface name="velocity"/>
-        <state_interface name="position">
-          <param name="initial_value">0.0</param>
-        </state_interface>
+        <!-- <command_interface name="status_request"/>
+        <command_interface name="maintenance_request"/> -->
+        <state_interface name="position"/>
         <state_interface name="velocity"/>
+        <state_interface name="motor_temperature"/>
+        <state_interface name="torque_current"/>
+        <!-- <state_interface name="status"/> -->
       </joint>
     </ros2_control>

File: src/description/ros2_control/drive/drive.rmd.ros2_control.xacro (robot description, xacro)
@@ -15,10 +15,16 @@
         <param name="joint_orientation">-1.0</param>
         <param name="operating_velocity">150</param> <!-- motor dps -->
-        <command_interface name="position"/>
+        <command_interface name="position" />
         <command_interface name="velocity"/>
+        <command_interface name="status_request"/>
+        <command_interface name="maintenance_request"/>
+        <command_interface name="maintenance_frame_high"/>
+        <command_interface name="maintenance_frame_low"/>
+        <command_interface name="maintenance_data_count"/>
         <state_interface name="position"/>
         <state_interface name="velocity"/>
         <state_interface name="motor_temperature"/>
         <state_interface name="torque_current"/>
+        <state_interface name="status"/>
       </joint>
       <joint name="propulsion_fr_joint">
@@ -27,10 +33,16 @@
         <param name="joint_orientation">1.0</param>
         <param name="operating_velocity">150</param> <!-- motor dps -->
-        <command_interface name="position"/>
+        <command_interface name="position" />
         <command_interface name="velocity"/>
+        <command_interface name="status_request"/>
+        <command_interface name="maintenance_request"/>
+        <command_interface name="maintenance_frame_high"/>
+        <command_interface name="maintenance_frame_low"/>
+        <command_interface name="maintenance_data_count"/>
         <state_interface name="position"/>
         <state_interface name="velocity"/>
         <state_interface name="motor_temperature"/>
         <state_interface name="torque_current"/>
+        <state_interface name="status"/>
       </joint>
       <joint name="propulsion_bl_joint">
@@ -39,10 +51,16 @@
         <param name="joint_orientation">1.0</param>
         <param name="operating_velocity">150</param> <!-- motor dps -->
-        <command_interface name="position"/>
+        <command_interface name="position" />
         <command_interface name="velocity"/>
+        <command_interface name="status_request"/>
+        <command_interface name="maintenance_request"/>
+        <command_interface name="maintenance_frame_high"/>
+        <command_interface name="maintenance_frame_low"/>
+        <command_interface name="maintenance_data_count"/>
         <state_interface name="position"/>
         <state_interface name="velocity"/>
         <state_interface name="motor_temperature"/>
         <state_interface name="torque_current"/>
+        <state_interface name="status"/>
       </joint>
       <joint name="propulsion_br_joint">
@@ -51,10 +69,16 @@
         <param name="joint_orientation">-1.0</param>
         <param name="operating_velocity">150</param> <!-- motor dps -->
-        <command_interface name="position"/>
+        <command_interface name="position" />
         <command_interface name="velocity"/>
+        <command_interface name="status_request"/>
+        <command_interface name="maintenance_request"/>
+        <command_interface name="maintenance_frame_high"/>
+        <command_interface name="maintenance_frame_low"/>
+        <command_interface name="maintenance_data_count"/>
         <state_interface name="position"/>
         <state_interface name="velocity"/>
         <state_interface name="motor_temperature"/>
         <state_interface name="torque_current"/>
+        <state_interface name="status"/>
       </joint>
     </ros2_control>

File: src/description/ros2_control/science/science.laser.ros2_control.xacro (robot description, xacro)
@@ -7,4 +7,7 @@
                 <param name="can_interface">${can_interface}</param>
                 <param name="can_id">0x130</param>
+                <param name="update_rate">10</param> <!-- Hz -->
+                <param name="logger_rate">5</param> <!-- Hz -->
+                <param name="logger_state">0</param> <!-- 0 for off, 1 for on -->
             </hardware>
             <gpio name="${name}">
@@ -12,5 +15,7 @@
                 <state_interface name="temperature"/>
                 <state_interface name="is_connected"/>
+                <state_interface name="status"/>
                 <command_interface name="laser_command"/>
+                <command_interface name="status_request"/>
             </gpio>
         </ros2_control>
