Commit message: HWI Upgrades (#110)
* changed broadcaster to controller and included other telemetry information

* odrive upgrades

* added request services

* included status decoding in RMDs

* decode error value and warn/error out depending on response

* reformatted rmd HWI

* saving some one shot progress

* encoding and decoding across command interfaces seems to be working

* holy fucking shit it works. Need to implement Torque control and then start doing doing this implementation on the rest of the HWIs

* updated smc hwi, issue with servo hwi

* fixed state issue, accepts all state interfaces and filters accordingly

* saving progress, killswitch seems to not be sending can messages for some reason

* saving changes, for some reason I cant see power module can commands being sent

* Power module and SMCs seem to be working, initial implementation of LED HWI created

* led hwi looks like its working

* added limit switch and rotary encoder HWI, included all necessary HWIs, needs fixing

* fixed motor status controller, manually choose command and state interfaces if default don't apply

* 3dof specific fixes

* motor status controller includes gpios, removing unnecessary gpio controllers

* Added DC Motor HWI

* Small changes to DC Motor HWI

* Fixing HWI issue

* Small Fix

* First test for steppers

* Moved revised athena_science code to monorepo

* Fixing Science Controller + HWI Templates for Steppers & Servos

* Restore accidentally deleted science.mock.ros2_control.xacro

* stepper stuff like kinda works??

* implemented and tested in virtual can servo, stepper, and dc HWIs

* working arm and steppers/DC motors

* WORKING DRIVE AND ARM

* quick fixes (joystick_index not set and removing /vscode and .codex

---------

Co-authored-by: duttaishan01 <duttaishan01@FIGARO.myguest.virtualbox.org>
Co-authored-by: HGardiner1 <henrygdnr@gmail.com>
Co-authored-by: UMDLoop Jetson Orin NX <umdloop@gmail.com>

File: src/description/ros2_control/science/science.servo.ros2_control.xacro (robot description, xacro)
@@ -7,5 +7,5 @@
                 <param name="update_rate">20</param> <!-- Hz -->
                 <param name="logger_rate">5</param> <!-- Hz -->
-                <param name="logger_state">1</param> <!-- 0 for off, 1 for on -->
+                <param name="logger_state">0</param> <!-- 0 for off, 1 for on -->
                 <param name="can_interface">can0</param>
                 <param name="can_id">0x80</param>
@@ -20,6 +20,12 @@
                 <command_interface name="position"/>
                 <command_interface name="velocity"/>
+                <command_interface name="status_request"/>
+                <command_interface name="maintenance_request"/>
+                <command_interface name="maintenance_frame_high"/>
+                <command_interface name="maintenance_frame_low"/>
+                <command_interface name="maintenance_data_count"/>
                 <state_interface name="position"/>
                 <state_interface name="velocity"/>
+                <state_interface name="status"/>
             </joint>
             <joint name="servo_rack_and_pinion_r">
@@ -32,6 +38,12 @@
                 <command_interface name="position"/>
                 <command_interface name="velocity"/>
+                <command_interface name="status_request"/>
+                <command_interface name="maintenance_request"/>
+                <command_interface name="maintenance_frame_high"/>
+                <command_interface name="maintenance_frame_low"/>
+                <command_interface name="maintenance_data_count"/>
                 <state_interface name="position"/>
                 <state_interface name="velocity"/>
+                <state_interface name="status"/>
             </joint>
             <joint name="servo_scoop_a">
@@ -43,5 +55,12 @@
                 <command_interface name="position"/>
                 <command_interface name="velocity"/>
+                <command_interface name="status_request"/>
+                <command_interface name="maintenance_request"/>
+                <command_interface name="maintenance_frame_high"/>
+                <command_interface name="maintenance_frame_low"/>
+                <command_interface name="maintenance_data_count"/>
                 <state_interface name="position"/>
+                <state_interface name="velocity"/>
+                <state_interface name="status"/>
             </joint>
             <joint name="servo_scoop_b">
@@ -53,5 +72,12 @@
                 <command_interface name="position"/>
                 <command_interface name="velocity"/>
+                <command_interface name="status_request"/>
+                <command_interface name="maintenance_request"/>
+                <command_interface name="maintenance_frame_high"/>
+                <command_interface name="maintenance_frame_low"/>
+                <command_interface name="maintenance_data_count"/>
                 <state_interface name="position"/>
+                <state_interface name="velocity"/>
+                <state_interface name="status"/>
             </joint>
             <joint name="servo_sampler_lift_l">
@@ -64,6 +90,12 @@
                 <command_interface name="position"/>
                 <command_interface name="velocity"/>
+                <command_interface name="status_request"/>
+                <command_interface name="maintenance_request"/>
+                <command_interface name="maintenance_frame_high"/>
+                <command_interface name="maintenance_frame_low"/>
+                <command_interface name="maintenance_data_count"/>
                 <state_interface name="position"/>
                 <state_interface name="velocity"/>
+                <state_interface name="status"/>
             </joint>
             <joint name="servo_sampler_lift_r">
@@ -76,6 +108,12 @@
                 <command_interface name="position"/>
                 <command_interface name="velocity"/>
+                <command_interface name="status_request"/>
+                <command_interface name="maintenance_request"/>
+                <command_interface name="maintenance_frame_high"/>
+                <command_interface name="maintenance_frame_low"/>
+                <command_interface name="maintenance_data_count"/>
                 <state_interface name="position"/>
                 <state_interface name="velocity"/>
+                <state_interface name="status"/>
             </joint>
             <joint name="servo_auger_lift">
@@ -88,5 +126,12 @@
                 <command_interface name="position"/>
                 <command_interface name="velocity"/>
+                <command_interface name="status_request"/>
+                <command_interface name="maintenance_request"/>
+                <command_interface name="maintenance_frame_high"/>
+                <command_interface name="maintenance_frame_low"/>
+                <command_interface name="maintenance_data_count"/>
                 <state_interface name="position"/>
+                <state_interface name="velocity"/>
+                <state_interface name="status"/>
             </joint>
         </ros2_control>

File: src/description/ros2_control/science/science.stepper.ros2_control.xacro (robot description, xacro)
@@ -5,28 +5,41 @@
             <hardware>
                 <plugin>stepper_ros2_control/STEPPERHardwareInterface</plugin>
+                <param name="update_rate">10</param> <!-- Hz -->
+                <param name="logger_rate">5</param> <!-- Hz -->
+                <param name="logger_state">0</param> <!-- 0 for off, 1 for on -->
+                <param name="can_interface">can0</param>
+                <param name="can_id">0x90</param>
             </hardware>
             <joint name="stepper_motor_a">
+                <param name="node_id">0x0</param>
+                <param name="gear_ratio">1</param>
+                <param name="rated_max">20</param>
+                <param name="joint_type">continuous</param>
                 <command_interface name="position"/>
                 <command_interface name="velocity"/>
+                <command_interface name="status_request"/>
+                <command_interface name="maintenance_request"/>
+                <command_interface name="maintenance_frame_high"/>
+                <command_interface name="maintenance_frame_low"/>
+                <command_interface name="maintenance_data_count"/>
                 <state_interface name="position"/>
-                <param name="initial_position">0.0</param>
                 <state_interface name="velocity"/>
-                <state_interface name="motor_temperature"/>
-                <state_interface name="torque_current"/>
-                <param name="gear_ratio">1</param>
-                <!-- TEMPORARY PARAMETERS -->
-                <param name="joint_orientation">1</param>
+                <state_interface name="status"/>
             </joint>
             <joint name="stepper_motor_b">
+                <param name="node_id">0x1</param>
+                <param name="gear_ratio">1</param>
+                <param name="rated_max">20</param>
+                <param name="joint_type">continuous</param>
                 <command_interface name="position"/>
                 <command_interface name="velocity"/>
+                <command_interface name="status_request"/>
+                <command_interface name="maintenance_request"/>
+                <command_interface name="maintenance_frame_high"/>
+                <command_interface name="maintenance_frame_low"/>
+                <command_interface name="maintenance_data_count"/>
                 <state_interface name="position"/>
-                <param name="initial_position">0.0</param>
                 <state_interface name="velocity"/>
-                <state_interface name="motor_temperature"/>
-                <state_interface name="torque_current"/>
-                <param name="gear_ratio">1</param>
-                <!-- TEMPORARY PARAMETERS -->
-                <param name="joint_orientation">1</param>
+                <state_interface name="status"/>
             </joint>
         </ros2_control>

File: src/description/ros2_control/science/science.talon.ros2_control.xacro (robot description, xacro)
@@ -30,8 +30,10 @@
         <command_interface name="position"/>
         <command_interface name="velocity"/>
+        <command_interface name="status_request"/>
         <state_interface name="position"/>
         <state_interface name="velocity"/>
         <state_interface name="motor_temperature"/>
         <state_interface name="torque_current"/>
+        <state_interface name="status"/>
       </joint>
       <joint name="talon_scoop">
@@ -49,8 +51,10 @@
         <command_interface name="position"/>
         <command_interface name="velocity"/>
+        <command_interface name="status_request"/>
         <state_interface name="position"/>
         <state_interface name="velocity"/>
         <state_interface name="motor_temperature"/>
         <state_interface name="torque_current"/>
+        <state_interface name="status"/>
       </joint>
     </ros2_control>

File: src/description/urdf/athena_arm.urdf.xacro (robot description, xacro)
@@ -25,4 +25,9 @@
   <!-- Import servo ros2_control description -->
   <xacro:include filename="$(find description)/ros2_control/arm/arm.servo.ros2_control.xacro" />
+  <!-- Import rotary encoder ros2_control description -->
+  <xacro:include filename="$(find description)/ros2_control/arm/arm.rotary_encoder.ros2_control.xacro" />
+  <!-- Import limit switch ros2_control descriptions -->
+  <xacro:include filename="$(find description)/ros2_control/arm/arm.base_limit_switch.ros2_control.xacro" />
+  <xacro:include filename="$(find description)/ros2_control/arm/arm.end_effector_limit_switch.ros2_control.xacro" />
   <!-- Import odrive ros2_control description -->
   <!-- <xacro:include filename="$(find description)/config/odrive.ros2_control.xacro" /> -->
@@ -45,4 +50,7 @@
     <xacro:rmd_ros2_control name="rmd"/>
     <xacro:servo_ros2_control name="servo"/>
+    <xacro:rotary_encoder_ros2_control name="rotary_encoder"/>
+    <xacro:base_arm_limit_switch_ros2_control name="base_arm_limit_switch"/>
+    <xacro:end_effector_limit_switch_ros2_control name="end_effector_limit_switch"/>
     <!-- <xacro:odrive_ros2_control name="odrive"/> -->
   </xacro:unless>

File: src/description/urdf/athena_drive.urdf.xacro (robot description, xacro)
@@ -7,4 +7,5 @@
   <xacro:arg name="sim_gazebo" default="true"/>
   <xacro:arg name="simulation_controllers" default=""/>
+  <xacro:arg name="deactivate_odrive" default="false"/>
   <xacro:include filename="$(find description)/urdf/athena_drive/athena_drive_macro.xacro"/>
   <xacro:include filename="$(find description)/urdf/athena_drive/athena_drive_macro.ros2_control.xacro"/>
@@ -28,6 +29,6 @@
   <!-- Import LED ros2_control description -->
   <xacro:include filename="$(find description)/ros2_control/drive/drive.led.ros2_control.xacro" />
-  <!-- Import killswitch ros2_control description -->
-  <xacro:include filename="$(find description)/ros2_control/drive/drive.killswitch.ros2_control.xacro" />
+  <!-- Import power_module ros2_control description -->
+  <xacro:include filename="$(find description)/ros2_control/drive/drive.power_module.ros2_control.xacro" />
   <!-- Contains description of drive -->
   <xacro:description/>
@@ -52,10 +53,12 @@
   </xacro:if>
   <xacro:unless value="$(arg use_mock_hardware)">
-    <xacro:odrive_ros2_control name="odrive"/>
+    <!-- ODrives-->
+    <xacro:odrive_ros2_control name="odrive" deactivate_odrive="$(arg deactivate_odrive)"/>
+    <!-- RMD -->
     <xacro:rmd_ros2_control name="rmd"/>
     <!-- LED status indicator (GPIO-based) -->
-    <xacro:led_ros2_control name="status_led" gpio_pin="25"/>
-    <!-- Killswitch (CAN-based) -->
-    <xacro:killswitch_ros2_control name="drive_killswitch"/>
+    <xacro:led_ros2_control name="drive_led" can_interface="can0"/>
+    <!-- PowerModule (CAN-based) -->
+    <xacro:power_module_ros2_control name="drive_power_module" can_interface="can0"/>
   </xacro:unless>
 </robot>

File: src/description/urdf/athena_science.urdf.xacro (robot description, xacro)
@@ -5,8 +5,11 @@
   <xacro:arg name="deactivate_talon" default="false"/>
   <xacro:include filename="$(find description)/ros2_control/science/science.mock.ros2_control.xacro"/>
-  <xacro:include filename="$(find description)/ros2_control/science/science.stepper.ros2_control.xacro" />
-  <xacro:include filename="$(find description)/ros2_control/science/science.servo.ros2_control.xacro" />
+  <xacro:include filename="$(find description)/ros2_control/science/science.stepper.ros2_control.xacro"/>
+  <xacro:include filename="$(find description)/ros2_control/science/science.servo.ros2_control.xacro"/>
+  <xacro:include filename="$(find description)/ros2_control/science/science.dc.ros2_control.xacro"/>
   <xacro:include filename="$(find description)/ros2_control/science/science.talon.ros2_control.xacro"/>
   <xacro:include filename="$(find description)/ros2_control/science/science.laser.ros2_control.xacro"/>
+  <xacro:include filename="$(find description)/ros2_control/science/science.led.ros2_control.xacro"/>
+  <xacro:include filename="$(find description)/ros2_control/science/science.limit_switch.ros2_control.xacro"/>
   <!-- create link fixed to the "world" -->
   <link name="world"/>
@@ -22,8 +25,13 @@
     <!-- Import servo ros2_control description -->
     <xacro:servo_ros2_control name="servo"/>
+    <!-- Import dc ros2_control description -->
+    <xacro:dc_ros2_control name="dc"/>
     <!-- Import talon ros2_control description -->
-    <xacro:talon_ros2_control name="talon" deactivate_talon="$(arg deactivate_talon)"/>
+    <!-- <xacro:talon_ros2_control name="talon" deactivate_talon="$(arg deactivate_talon)"/> -->
     <!-- Import laser ros2_control description (CAN-based) -->
     <xacro:laser_ros2_control name="spectrometry_laser"/>
+    <!-- Import LED and limit switch ros2_control descriptions -->
+    <xacro:science_led_ros2_control name="fluoro_led_hwi"/>
+    <xacro:science_limit_switch_ros2_control name="science_limit_switch_hwi"/>
   </xacro:unless>
 </robot>
